File: Sentry_Turret.kicad_pcb (KiCad board)
At the start: 2 copper layers, 104 x 60 mm, 36 parts, among them J14 501645-1620, J16 172298-1108

Commit message: Check for jed
Parts:
- added L_Light1: Conn_01x02_Pin, Connector_AMASS:AMASS_XT30U-F_1x02_P5.0mm_Vertical, F.Cu at (56.9, 74.5)
- added R_Light1: Conn_01x02_Pin, Connector_AMASS:AMASS_XT30U-F_1x02_P5.0mm_Vertical, F.Cu at (92.0, 74.5)
- moved J14 18.8 mm to (75.5, 53.5), turned to 180 degrees
- moved J16 16.6 mm to (69.5, 69.5)
- moved L_CAN_Yaw1 9.43 mm to (48.9, 48.3), turned to 90 degrees
- moved R_CAN_Yaw1 9.34 mm to (100.7, 48.3), turned to -90 degrees
- moved UART_Orin1 7.97 mm to (92.0, 58.2), turned to 0 degrees
- moved SWD_In_Orin1 7.91 mm to (57.2, 58.2), turned to 0 degrees
- moved R_PWR_Yaw1 3.02 mm to (120.0, 44.3)
- moved L_PWR_Pitch1 2.97 mm to (27.6, 60.6)
- moved L_PWR_Yaw1 2.97 mm to (27.6, 39.3)
- moved L_PWR_Agitator1 2.79 mm to (39.5, 77.6)
- moved R_PWR_Agitator1 2.79 mm to (104.5, 77.6)
- moved R_PWR_TFly1 2.29 mm to (120.0, 65.6)
- moved L_PWR_BFly1 0.71 mm to (41.0, 27.6)
- moved L_PWR_TFly1 0.71 mm to (59.0, 27.6)
- moved PWR_Orin1 0.71 mm to (77.0, 27.6)
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- renumbered L_+PWR_Agitator1 to L_PWR_Agitator1
Routing:
- net /CAN2-: track 0.00 -> 70.9 mm
- net /CAN2+: track 0.00 -> 69.5 mm

Commit message: Layout review
Parts:
- added G***: LOGO, Robomaster_Special:StampedeLogo, F.Cu at (86.0, 39.4)
- added Ref_Out2: Conn_01x04_Pin, Connector_JST:JST_GH_BM04B-GHS-TBT_1x04-1MP_P1.25mm_Vertical, F.Cu at (102.0, 50.6)
- moved D1 123.1 mm to (27.7, 54.3)
- moved R1 123.0 mm to (27.6, 51.2)
- moved R3 89.7 mm to (65.4, 32.3), turned to 90 degrees
- moved D3 88.8 mm to (65.4, 28.0), turned to -90 degrees
- moved D2 68.1 mm to (85.6, 70.4), turned to 180 degrees
- moved R2 66.9 mm to (85.6, 73.6), turned to 180 degrees
- moved R_PWR_Pitch1 49.5 mm to (107.5, 75.5), turned to 0 degrees
- moved L_Light1 45.8 mm to (27.6, 39.3), turned to -90 degrees
- moved L_PWR_Yaw1 43.8 mm to (52.3, 75.5), turned to 0 degrees
- moved R_PWR_TFly1 43.4 mm to (95.0, 30.1), turned to 180 degrees
- moved R_PWR_Yaw1 42.3 mm to (91.4, 75.5), turned to 0 degrees
- moved R_Light1 42.2 mm to (121.5, 44.3)
- moved R_CAN_Pitch1 34.3 mm to (107.0, 67.1), turned to 90 degrees
- moved UART_Orin1 25.9 mm to (74.4, 39.1)
- moved Ref_Out1 21.8 mm to (92.6, 50.6), turned to -90 degrees
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Connections:
- J16 pad 1: /Shooter_{GND} -> unconnected-(J16-Pad1)
- J16 pad 3: /OrinPWR_{GND} -> /Shooter_{GND}
- J16 pad 4: unconnected-(J16-Pad4) -> /OrinPWR_{GND}
- J16 pad 5: /Shooter_{+24V} -> unconnected-(J16-Pad5)
- J16 pad 7: /OrinPWR_{+19V} -> /Shooter_{+24V}
- J16 pad 8: unconnected-(J16-Pad8) -> /OrinPWR_{+19V}
Routing:
- net /CAN2-: track 70.9 -> 205.2 mm
- net /CAN2+: track 69.5 -> 201.5 mm
- net /CAN1+: track 0.00 -> 75.5 mm
- net /CAN1-: track 0.00 -> 74.8 mm
- net /Ref_{PWR}: track 0.00 -> 29.4 mm
- net /Ref_{CAN}+: track 0.00 -> 26.3 mm
- net /Ref_{CAN}-: track 0.00 -> 23.5 mm
- net /Ref_{GND}: track 0.00 -> 19.7 mm
- net /SWD_{GND}: track 0.00 -> 13.7 mm
- net /SWD_{3V3}: track 0.00 -> 13.2 mm
- net /OrinPWR_{+19V}: track 0.00 -> 12.8 mm
- net /UART_{3V3}: track 0.00 -> 11.3 mm
- net /SWD_{SWDIO}: track 0.00 -> 11.0 mm
- net /UART_{RX}: track 0.00 -> 11.0 mm
- net /SWD_{SWCLK}: track 0.00 -> 10.7 mm
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- added copper zone on F.Cu, net /Gimbal_{+24V}
- added copper zone on B.Cu, net /Gimbal_{GND}
- added copper zone on B.Cu, net /OrinPWR_{+19V}
- added copper zone on B.Cu, net /OrinPWR_{GND}
- added copper zone on F.Cu, net /Shooter_{+24V}
Other:
- board text added: "GIMB PWR"
- board text added: "ORIN PWR"
- board text added: "SHTR PWR"
- board text added: "UT Stampede Sentry Turret Board Morris Lin"

Commit message: Finalized board for order
Parts:
- moved J14 6.48 mm to (69.4, 50.2)
- moved SWD_In_Orin1 4.85 mm to (50.5, 50.2)
- moved Ref_Out1 3.35 mm to (89.2, 50.6)
- moved Ref_Out2 0.20 mm to (101.8, 50.6)
Routing:
- net /Ref_{CAN}-: track 23.5 -> 30.3 mm
- net /Ref_{CAN}+: track 26.3 -> 33.0 mm
- net /Ref_{PWR}: track 29.4 -> 35.8 mm
- net /Ref_{GND}: track 19.7 -> 26.0 mm
- net /CAN1+: track 75.5 -> 70.6 mm
- net /CAN1-: track 74.8 -> 69.9 mm
- net /CAN2-: track 205.2 -> 201.6 mm
- net /CAN2+: track 201.5 -> 197.8 mm
- net /SWD_{GND}: track 13.7 -> 12.0 mm
- net /SWD_{SWCLK}: track 10.7 -> 9.08 mm
- net /SWD_{3V3}: track 13.2 -> 11.6 mm
- net /SWD_{SWDIO}: track 11.0 -> 9.41 mm
- net /UART_{3V3}: track 11.3 -> 9.92 mm
- net /UART_{RX}: track 11.0 -> 9.84 mm
- net /UART_{TX}: track 10.7 -> 10.1 mm
